File: dshield.brd (EAGLE design)
At the start: 160 x 100 mm, 17 parts, among them IC1 LM1117DTX-3.3, IC2 LM1117DTX-3.3

Commit message: Add files via upload
Parts:
- added BTPL1, BTPL2, BTPL3, BTPL4, BTPL5, BTPL6, BTPL7, BTPL8: GS-SH-2XXT, goodsky_btpl:G_RELAY_SMD
- added C5, C6: (no value), rcl:E2,5-6
- added D1, D2, D3, D4, D5, D6, D7, D8: 1N4004, diode:DO41-10
- added IC3: 7805DT, linear:TO252
- added Q1, Q2, Q3, Q4, Q5, Q6, Q7, Q8: IRF520, transistor-power:TO220BV
- moved C4 206.8 mm to (-79.8, 34.9)
- moved C1 198.3 mm to (-60.8, 34.9)
- moved C2 195.7 mm to (-67.1, 34.9)
- moved C3 193.2 mm to (-73.5, 34.9)
- moved U$3 189.1 mm to (-84.2, -10.1), turned to 90 degrees
- moved IC1 176.5 mm to (-67.1, 24.8), turned to 180 degrees
- moved IC2 173.9 mm to (-76.0, 24.8), turned to 180 degrees
- moved DAC0 161.0 mm to (-110.3, 29.9)
- moved DAC1 161.0 mm to (-105.2, 29.9)
- moved U$2 156.0 mm to (-24.0, 42.3)
- moved U$4 152.8 mm to (-59.1, 52.2)
- moved U$1 143.0 mm to (-36.6, -0.60), flipped to the bottom, turned to 90 degrees
- moved SV1 113.7 mm to (-85.8, -54.6)
- moved SV2 111.2 mm to (-66.3, -54.6)
- moved SV3 108.7 mm to (-46.8, -54.6)
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Connections:
- new net 5V: BTPL1.C2, BTPL2.C2, BTPL3.C2, BTPL4.C2, BTPL5.C2, BTPL6.C2, BTPL7.C2, BTPL8.C2, C6.+, D1.C, D2.C, D3.C, D4.C, D5.C, D6.C, D7.C, D8.C, IC3.2
- new net D1: BTPL2.C1, D2.A, Q2.D
- new net D2: BTPL1.C1, D1.A, Q1.D
- new net D3: BTPL7.C1, D7.A, Q7.D
- new net D4: BTPL3.C1, D3.A, Q3.D
- new net D5: BTPL4.C1, D4.A, Q4.D
- new net D6: BTPL8.C1, D8.A, Q8.D
- new net D7: BTPL5.C1, D5.A, Q5.D
- new net D8: BTPL6.C1, D6.A, Q6.D
- new net N$1: Q1.G, Q2.G, Q3.G, Q4.G, Q5.G, Q6.G, Q7.G, Q8.G
- new net N$2: BTPL1.P1, BTPL2.P1, BTPL3.P1, BTPL4.P1, BTPL5.P1, BTPL6.P1, BTPL7.P1, BTPL8.P1
- new net N$3: BTPL1.NO1, BTPL2.NO1, BTPL3.NO1, BTPL4.NO1, BTPL5.NO1, BTPL6.NO1, BTPL7.NO1, BTPL8.NO1
- net 9V: now also C5.+, IC3.1
- net GND: now also C5.-, C6.-, IC3.3, Q1.S, Q2.S, Q3.S, Q4.S, Q5.S, Q6.S, Q7.S, Q8.S
Other:
- board size 160 x 100 mm -> 284 x 120 mm
